File: Project Course/Task 5/TeamB.brd (EAGLE design)
At the start: 76.2 x 69.5 mm, 33 parts, among them Q1 MIC29300-5.0WU, Q2 MIC29300-3.3WU, Q3 MIC29300-12WU, U0 26V, U1 26V, U2 5V, U3 3.3V, U4 12V

Commit message: Corrected Packages, Verified Trace widths
Used TE5 fuses, and verified everything using 1 oz copper
Parts:
- removed D1, D2, D3, D4: GREEN, led:CHIP-LED0805
- added LED1, LED2, LED3, LED4: GREEN, led:SML1206
- C1, C2, C3, C4, C5, C6: device TinyGadget(1):C025-025X050 -> rcl:C1206
- F_CPU: value 3.3V 1.5A -> 1.5A
- F_LIDAR: value 12V 3A -> 3A
- F_MAIN: value 27V 20A -> 20A
- F_MOT: value 27V 15A -> 15A
- F_WIFI: value 5V 1.5A -> 1.5A
- R1, R2, R3, R4: device resistor:R0402 -> rcl:R1206
- moved C3 3.59 mm to (40.6, 8.89), turned to 90 degrees
- moved C1 3.59 mm to (40.6, 41.9), turned to 90 degrees
- moved C2 3.59 mm to (40.6, 25.4), turned to 90 degrees
- moved C6 2.84 mm to (44.5, 11.4), turned to 270 degrees
- moved C4 2.84 mm to (44.5, 44.5), turned to 270 degrees
- moved C5 2.84 mm to (44.5, 27.9), turned to 270 degrees
- moved U1 2.54 mm to (50.8, 61.0)
- moved R1 1.27 mm to (21.6, 26.7)
- moved R2 1.27 mm to (21.6, 21.6)
- moved R3 1.27 mm to (21.6, 16.5)
- moved R4 1.27 mm to (21.6, 11.4)
Connections:
- net GND: now also LED1.C, LED2.C, LED3.C, LED4.C; no longer D1.C, D2.C, D3.C, D4.C
- net N$11: now also LED3.A, R3.1; no longer D2.A, R2.1
- net N$13: now also LED4.A; no longer D4.A
- net N$5: now also LED1.A; no longer D1.A
- net N$8: now also LED2.A, R2.1; no longer D3.A, R3.1
Routing:
- net N$12: track 122.6 -> 80.2 mm
- net N$1: track 75.1 -> 55.9 mm
- net GND: track 43.9 -> 61.5 mm, vias 2 -> 5
- net N$10: track 6.14 -> 0.00 mm
- net N$7: track 77.2 -> 73.3 mm
- net N$4: track 54.5 -> 52.5 mm
- net N$2: track 55.4 -> 54.6 mm
- added copper zone on layer 1, net GND
- added copper zone on layer 1, net N$1
- added copper zone on layer 1, net N$10
- added copper zone on layer 1, net N$12
Other:
- board text added: "Rev. 0.3"
- board text removed: "Rev. 0.1"
