File: Project Course/Task 10 Power Distribution Board/powerdist2.brd (EAGLE design)
At the start: 88.9 x 75.9 mm, 33 parts

Commit message: For voltage monitoring, I used a single header pin
Parts:
- removed CIN, COUT: CAPACITORTH_CAP, TinyGadget(1):C025-025X050
- removed CPU3.3V1A: MIC29150/29300/29500, Micrel-Voltage-Regulator:MIC29150/29300/29500
- removed ENCODER: C-GRID-02-70553, con-molex:70553-02
- removed TVS-MAIN4: 26V, Micrel-Voltage-Regulator:TVS-SMAJ
- added BAT_MON: TSW-101-02-S-S, con-samtec:TSW-101-02-S-S
- added CIN3, COUT3, DEC_CAP1, DEC_CAP1_2, DEC_CAP2, DEC_CAP2_2: CAPACITORTH_CAP, TinyGadget(1):C025-025X050
- added F_LID1, F_SERVO1: (no value), fuse:GSH15
- added LDO3, SERVO1: 5566-2, con-molex:5566-2
- added LED_LDO3, LED_SRV1: (no value), led:CHIP-LED0805
- added LID12V1A1: MIC29150/29300/29500, Micrel-Voltage-Regulator:MIC29150/29300/29500
- added PWR_SW, SRV1_SW, SRV2_SW: (no value), switch:REKN
- added RSRV1, R_LDO3, R_MON2: 2.2K, resistor:R0402
- added R_MON1: 3.0K, resistor:R0402
- added TVS_3.3: 16V, Micrel-Voltage-Regulator:TVS-SMAJ
- TVS-MAIN1: value 3.3V -> 16V
- moved TVS-MAIN1 182.5 mm to (-26.7, -120.7), turned to 0 degrees
- renumbered CPU to DUE, F_CPU to F_DUE, F_MOT to F_SERVO2, LEDLIDAR to LED_LDO2, LEDMOTOR to LED_SRV2, LEDWIFI_ENC to LED_LDO1, LIDAR to LDO2, MOTOR to SERVO2, R1 to RSRV2, R3 to R_LDO1, R4 to R_LDO2, WIFI to LDO1
Connections:
- new net N$14: F_SUP.1, PWR_SW.1A
- new net N$15: DEC_CAP1.1, DEC_CAP1_2.1, F_SERVO1.2, RSRV1.2, SERVO1.1
- new net N$16: LED_SRV1.A, RSRV1.1
- new net N$17: F_SERVO2.1, SRV2_SW.1A
- new net N$18: BAT_MON.1, R_MON1.1, R_MON2.2, TVS_3.3.CAT
- new net N$19: COUT3.1, F_LID1.1, LID12V1A1.VOUT
- new net N$20: CIN3.1, LID12V1A1.VIN
- new net N$21: F_LID1.2, LDO3.1, R_LDO3.2, TVS-MAIN1.CAT
- new net N$22: LED_LDO3.A, R_LDO3.1
- net GND: now also CIN3.2, COUT3.2, DEC_CAP1.2, DEC_CAP1_2.2, DEC_CAP2.2, DEC_CAP2_2.2, LDO3.2, LED_LDO3.C, LED_SRV1.C, LID12V1A1.GND, R_MON2.1, SERVO1.2, TVS_3.3.AN; no longer CIN.2, COUT.2, CPU3.3V1A.GND, ENCODER.2, TVS-MAIN4.AN
- net N$1: now also DEC_CAP2.1, DEC_CAP2_2.1; no longer TVS-MAIN4.CAT
- net N$10: now also PWR_SW.0A; no longer F_SUP.1
- net N$12: now also F_DUE.1, R_MON1.2, SRV1_SW.0A, SRV2_SW.0A; no longer CIN.1, CPU3.3V1A.VIN, F_SERVO2.1
- net N$3: now also F_SERVO1.1, SRV1_SW.1A; no longer COUT.1, CPU3.3V1A.VOUT, F_DUE.1
- net N$4: no longer TVS-MAIN1.CAT
- net N$7: no longer ENCODER.1
Routing:
- net N$12: track 19.7 -> 0.36 mm, vias 0 -> 1
- net N$4: track 8.20 -> 7.43 mm
- net N$10: track 1.69 -> 0.97 mm
- net N$3: track 0.36 -> 0.00 mm, vias 1 -> 0
