File: Project/Task10/powerdist2.brd (EAGLE design)
At the start: 88.9 x 75.9 mm, 50 parts

Commit message: Updated power distribution board schematic
Parts:
- removed LID12V1A, LID12V1A1, WIFI5V1A1: MIC29150/29300/29500, Micrel-Voltage-Regulator:MIC29150/29300/29500
- removed RSRV1, RSRV2, R_LDO1, R_LDO2, R_LDO3, R_MON2: 2.2K, resistor:R0402
- removed R_MON1: 3.0K, resistor:R0402
- removed TVS-MAIN: 26V, Micrel-Voltage-Regulator:TVS-SMAJ
- removed TVS-MAIN1, TVS-MAIN3, TVS_3.3: 16V, Micrel-Voltage-Regulator:TVS-SMAJ
- removed TVS-MAIN2: 5V, Micrel-Voltage-Regulator:TVS-SMAJ
- added BATT_A: 22-23-2021, con-molex:22-23-2021
- added D1: 3.3V Zener, Task5:SMA
- added R1, R3, R4, R5, R6: (no value), rcl:0309/10
- added R7: 3K, rcl:0309/10
- added R8: 2.2K, rcl:0309/10
- added U$1, U$6, U$7: MIC29150/29300/29500, Task5:TO220
- added U$2, U$3, U$4, U$5: TVS-DIODE-SMA, Task5:SMA
- BAT_MON: value TSW-101-02-S-S -> (none)
- F_DUE: value (none) -> 2A
- F_LID, F_LID1, F_WIFI: value (none) -> 5A
- F_SERVO1, F_SERVO2: value (none) -> 10A
- F_SUP: value (none) -> 20A
- R2: value 2.2K -> (none); device resistor:R0402 -> rcl:0309/10
- moved R2 212.6 mm to (-53.3, -174.0)
- renumbered INPUT_LIPO_7.4V to BATT_B
Connections:
- removed net N$12: CIN1.1, CIN2.1, F_DUE.1, F_SUP.2, LID12V1A.VIN, R_MON1.2, SRV1_SW.0A, SRV2_SW.0A, TVS-MAIN.CAT, WIFI5V1A1.VIN
- net GND: now also BATT_A.2, D1.AN, R8.1, U$1.2, U$2.AN, U$3.AN, U$4.AN, U$5.AN, U$6.2, U$7.2; no longer LID12V1A.GND, LID12V1A1.GND, R_MON2.1, TVS-MAIN.AN, TVS-MAIN1.AN, TVS-MAIN2.AN, TVS-MAIN3.AN, TVS_3.3.AN, WIFI5V1A1.GND
- net N$1: now also R2.2; no longer RSRV2.2
- net N$10: now also BATT_A.1
- net N$11: now also LEDCPU.A, R3.1; no longer LED_LDO1.A, R_LDO1.1
- net N$13: now also LED_LDO1.A, R4.1; no longer LED_LDO2.A, R_LDO2.1
- net N$15: now also R1.2; no longer RSRV1.2
- net N$16: now also LED_LDO2.A, R5.1; no longer LED_SRV1.A, RSRV1.1
- net N$18: now also D1.CAT, R7.1, R8.2; no longer R_MON1.1, R_MON2.2, TVS_3.3.CAT
- net N$19: now also U$1.3; no longer LID12V1A1.VOUT
- net N$2: now also R5.2, U$4.CAT; no longer R_LDO2.2, TVS-MAIN3.CAT
- net N$20: now also CIN1.1, CIN2.1, F_DUE.1, F_SUP.2, R7.2, SRV1_SW.0A, SRV2_SW.0A, U$1.1, U$2.CAT, U$6.1, U$7.1; no longer LID12V1A1.VIN
- net N$21: now also R6.2, U$3.CAT; no longer R_LDO3.2, TVS-MAIN1.CAT
- net N$22: now also R6.1; no longer R_LDO3.1
- net N$4: now also R3.2; no longer R2.2
- net N$5: now also LED_SRV1.A, R1.1; no longer LED_SRV2.A, RSRV2.1
- net N$6: now also U$7.3; no longer WIFI5V1A1.VOUT
- net N$7: now also R4.2, U$5.CAT; no longer R_LDO1.2, TVS-MAIN2.CAT
- net N$8: now also LED_SRV2.A; no longer LEDCPU.A
- net N$9: now also U$6.3; no longer LID12V1A.VOUT
Routing:
- net N$8: track 3.38 -> 0.00 mm
- net N$5: track 3.38 -> 0.00 mm
- net N$13: track 3.38 -> 0.00 mm
- net N$11: track 3.38 -> 0.00 mm
- net N$20: track 0.00 -> 0.36 mm, vias 0 -> 1
- net N$12: track 0.36 -> 0.00 mm, vias 1 -> 0

Commit message: Updated Schematic, ready for submitting...
Parts:
- removed PWR_SW, SRV1_SW, SRV2_SW: (no value), switch:REKN
- added S1: (no value), switch:255SB
- ACC2, ACC3, SERVO1, SERVO2: value 5566-2 -> (none)
- C1, C2: value CAPACITORTH_CAP -> (none)
- R1, R2, R3, R4, R5, R6: value (none) -> 1K
- U$2: value TVS-DIODE-SMA -> 8V
- renumbered DEC_CAP1 to C1, DEC_CAP1_2 to C2, DEC_CAP2 to C3, DEC_CAP2_2 to C4, LDO1 to ACC1, LDO2 to ACC2, LDO3 to ACC3, LEDCPU to LED4, LED_LDO1 to LED1, LED_LDO2 to LED2, LED_LDO3 to LED3, LED_SRV1 to LED6, LED_SRV2 to LED5
Connections:
- removed net N$17: F_SERVO2.1, SRV2_SW.1A
- removed net N$20: CIN1.1, CIN2.1, CIN3.1, F_DUE.1, F_SUP.2, R7.2, SRV1_SW.0A, SRV2_SW.0A, U$1.1, U$2.CAT, U$6.1, U$7.1
- removed net N$3: F_SERVO1.1, SRV1_SW.1A
- new net V_SUPPLY: CIN1.1, CIN2.1, CIN3.1, F_DUE.1, F_SERVO1.1, F_SERVO2.1, F_SUP.2, R7.2, U$1.1, U$2.CAT, U$6.1, U$7.1
- net N$10: now also S1.2; no longer PWR_SW.0A
- net N$14: now also S1.1; no longer PWR_SW.1A
Routing:
- net N$20: track 0.36 -> 0.00 mm, vias 1 -> 0
