File: Project/Task10/PDM.sch (EAGLE design)
At the start: 43 parts

Commit message: Fixed Capacitors and Schematic
Parts:
- added PAD1: (no value), wirepad:2,15/1,0
- C2, C4: value CAPACITORTH_CAP -> (none); device TinyGadget(1):CAPACITORTH_CAP -> rcl:CPOL-USTT5D11
- F_BATT: value 20A -> 15A
- F_SERVO1, F_SERVO2: value 10A -> 7.5A
Connections:
- net GND: now also C2.-, C4.-; no longer C2.2, C4.2
- net N$1: now also C4.+; no longer C4.1
- net N$15: now also C2.+; no longer C2.1
Changed lines of the file:
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@@
 <part name="SUPPLY2" library="supply2" deviceset="GND" device=""/>
 <part name="BAT_MON" library="con-samtec" deviceset="TSW-101-02-S-S" device="" value=""/>
-<part name="C2" library="TinyGadget(1)" deviceset="CAPACITOR" device="TH_CAP" value=""/>
-<part name="C4" library="TinyGadget(1)" deviceset="CAPACITOR" device="TH_CAP"/>
 <part name="SUPPLY8" library="supply2" deviceset="GND" device=""/>
 <part name="ACC3" library="con-molex" deviceset="5566-2" device="" value=""/>
@@
 <part name="U$2" library="MRSDTeamB" deviceset="MIC29150/29300/29500" device="HORIZONTAL"/>
 <part name="U$3" library="MRSDTeamB" deviceset="MIC29150/29300/29500" device="HORIZONTAL"/>
-<part name="F_BATT" library="MRSDTeamB" deviceset="FUSE-" device="ATO" value="20A"/>
+<part name="F_BATT" library="MRSDTeamB" deviceset="FUSE-" device="ATO" value="15A"/>
 <part name="F_DUE" library="MRSDTeamB" deviceset="FUSE-" device="ATO" value="2A"/>
-<part name="F_SERVO1" library="MRSDTeamB" deviceset="FUSE-" device="ATO" value="10A"/>
-<part name="F_SERVO2" library="MRSDTeamB" deviceset="FUSE-" device="ATO" value="10A"/>
+<part name="F_SERVO1" library="MRSDTeamB" deviceset="FUSE-" device="ATO" value="7.5A"/>
+<part name="F_SERVO2" library="MRSDTeamB" deviceset="FUSE-" device="ATO" value="7.5A"/>
 <part name="ACC1" library="con-molex" deviceset="5566-2" device="" value=""/>
+<part name="C2" library="rcl" deviceset="CPOL-US" device="TT5D11"/>
+<part name="C4" library="rcl" deviceset="CPOL-US" device="TT5D11"/>
+<part name="PAD1" library="wirepad" deviceset="2,15/1,0" device=""/>
 </parts>
 <sheets>
@@
 <instance part="SUPPLY2" gate="GND" x="35.56" y="109.22"/>
 <instance part="BAT_MON" gate="-1" x="62.23" y="121.92"/>
-<instance part="C2" gate="G$1" x="149.86" y="139.7" smashed="yes">
-<attribute name="NAME" x="153.416" y="137.795" size="1.778" layer="95"/>
-</instance>
-<instance part="C4" gate="G$1" x="149.86" y="109.22" smashed="yes">
-<attribute name="NAME" x="153.416" y="107.315" size="1.778" layer="95"/>
-</instance>
 <instance part="SUPPLY8" gate="GND" x="256.54" y="104.14"/>
 <instance part="ACC3" gate="-1" x="297.18" y="116.84"/>
@@
 <instance part="ACC1" gate="-1" x="297.18" y="180.34"/>
 <instance part="ACC1" gate="-2" x="297.18" y="177.8"/>
+<instance part="C2" gate="G$1" x="149.86" y="137.16"/>
+<instance part="C4" gate="G$1" x="149.86" y="106.68"/>
+<instance part="PAD1" gate="1" x="53.34" y="134.62"/>
 </instances>
 <busses>
@@
 <pinref part="LED5" gate="G$1" pin="C"/>
 <wire x1="152.4" y1="101.6" x2="149.86" y2="101.6" width="0.1524" layer="91"/>
+<pinref part="C4" gate="G$1" pin="-"/>
 <junction x="149.86" y="101.6"/>
-<pinref part="C4" gate="G$1" pin="2"/>
-<wire x1="149.86" y1="104.14" x2="149.86" y2="101.6" width="0.1524" layer="91"/>
 </segment>
 <segment>
@@
 <segment>
 <pinref part="SUPPLY16" gate="GND" pin="GND"/>
+<pinref part="C2" gate="G$1" pin="-"/>
 <pinref part="LED6" gate="G$1" pin="C"/>
-<wire x1="152.4" y1="132.08" x2="149.86" y2="132.08" width="0.1524" layer="91"/>
+<wire x1="149.86" y1="132.08" x2="152.4" y2="132.08" width="0.1524" layer="91"/>
 <junction x="149.86" y="132.08"/>
-<pinref part="C2" gate="G$1" pin="2"/>
-<wire x1="149.86" y1="134.62" x2="149.86" y2="132.08" width="0.1524" layer="91"/>
 </segment>
 <segment>
@@
 <net name="N$1" class="0">
 <segment>
-<wire x1="147.32" y1="111.76" x2="149.86" y2="111.76" width="0.1524" layer="91"/>
-<pinref part="C4" gate="G$1" pin="1"/>
-<wire x1="149.86" y1="111.76" x2="162.56" y2="111.76" width="0.1524" layer="91"/>
-<junction x="149.86" y="111.76"/>
 <pinref part="R2" gate="G$1" pin="2"/>
 <pinref part="SERVO2" gate="-1" pin="S"/>
 <wire x1="162.56" y1="111.76" x2="170.18" y2="111.76" width="0.1524" layer="91"/>
+<pinref part="F_SERVO2" gate="G$1" pin="2"/>
+<wire x1="162.56" y1="111.76" x2="149.86" y2="111.76" width="0.1524" layer="91"/>
 <junction x="162.56" y="111.76"/>
-<pinref part="F_SERVO2" gate="G$1" pin="2"/>
+<pinref part="C4" gate="G$1" pin="+"/>
+<wire x1="149.86" y1="111.76" x2="147.32" y2="111.76" width="0.1524" layer="91"/>
+<wire x1="149.86" y1="109.22" x2="149.86" y2="111.76" width="0.1524" layer="91"/>
+<junction x="149.86" y="111.76"/>
 </segment>
 </net>
@@
 <segment>
 <pinref part="SERVO1" gate="-1" pin="S"/>
-<wire x1="147.32" y1="142.24" x2="149.86" y2="142.24" width="0.1524" layer="91"/>
-<pinref part="C2" gate="G$1" pin="1"/>
-<wire x1="149.86" y1="142.24" x2="162.56" y2="142.24" width="0.1524" layer="91"/>
-<junction x="149.86" y="142.24"/>
 <pinref part="R1" gate="G$1" pin="2"/>
 <wire x1="162.56" y1="142.24" x2="170.18" y2="142.24" width="0.1524" layer="91"/>
+<pinref part="F_SERVO1" gate="G$1" pin="2"/>
+<wire x1="147.32" y1="142.24" x2="149.86" y2="142.24" width="0.1524" layer="91"/>
 <junction x="162.56" y="142.24"/>
-<pinref part="F_SERVO1" gate="G$1" pin="2"/>
-</segment>
-</net>
+<pinref part="C2" gate="G$1" pin="+"/>
+<wire x1="149.86" y1="142.24" x2="162.56" y2="142.24" width="0.1524" layer="91"/>
+<wire x1="149.86" y1="139.7" x2="149.86" y2="142.24" width="0.1524" layer="91"/>
+<junction x="149.86" y="142.24"/>
+</segment>
+</net>
