File: Project/Task10/PDM.brd (EAGLE design)
At the start: 101.3 x 76.2 mm, 43 parts

Commit message: Task 10 ready to submit
Parts:
- R7: value 3K -> 15.4K
- R8: value 2.2K -> 10K
- U1, U2, U3: value MIC29150/29300/29500VERTICAL -> (none)
- renumbered U$1 to U1, U$2 to U2, U$3 to U3
Other:
- board text added: "Rev 0.2"
- board text removed: "Rev 0.1"
Changed lines of the file:
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@@
 <wire x1="76.2" y1="7.62" x2="76.2" y2="35.56" width="0.4064" layer="21"/>
 <text x="50.8" y="2.54" size="1.778" layer="25">MRSD Team B, Fall 2013</text>
-<text x="85.09" y="2.54" size="1.778" layer="25">Rev 0.1</text>
+<text x="85.09" y="2.54" size="1.778" layer="25">Rev 0.2</text>
 </plain>
 <attributes>
@@
 <attribute name="NAME" x="73.66" y="10.16" size="1.27" layer="25" rot="R180"/>
 </element>
-<element name="R7" library="rcl" package="R1206" value="3K" x="60.96" y="34.29" rot="R90"/>
-<element name="R8" library="rcl" package="R1206" value="2.2K" x="60.96" y="24.13" rot="R90"/>
+<element name="R7" library="rcl" package="R1206" value="15.4K" x="60.96" y="34.29" rot="R90"/>
+<element name="R8" library="rcl" package="R1206" value="10K" x="60.96" y="24.13" rot="R90"/>
 <element name="C5" library="rcl" package="C1206K" value="10uF" x="52.07" y="41.91" smashed="yes" rot="R90">
 <attribute name="NAME" x="50.97" y="40.945" size="1.016" layer="25" rot="R90"/>
@@
 <element name="F_BATT" library="MRSDTeamB" package="ATO" value="15A" x="15.24" y="16.51" smashed="yes" rot="R180">
 <attribute name="VALUE" x="21.08" y="22.41" size="1.27" layer="21" rot="R180"/>
-<attribute name="NAME" x="14.83" y="22.07" size="1.27" layer="21" rot="R180"/>
+<attribute name="NAME" x="14.83" y="22.705" size="1.27" layer="21" rot="R180"/>
 </element>
 <element name="F_DUE" library="MRSDTeamB" package="ATO" value="2A" x="41.91" y="35.56" smashed="yes" rot="R90">
@@
 <element name="BATT1_W" library="MRSDTeamB" package="CON_XT60_PIGTAIL" value="" x="52.07" y="19.05" rot="R180"/>
 <element name="BATT2_W" library="MRSDTeamB" package="CON_XT60_PIGTAIL" value="" x="52.07" y="13.97" rot="R180"/>
-<element name="U$1" library="MRSDTeamB" package="TO220V" value="MIC29150/29300/29500VERTICAL" x="54.61" y="43.18" smashed="yes" rot="R90"/>
-<element name="U$2" library="MRSDTeamB" package="TO220V" value="MIC29150/29300/29500VERTICAL" x="69.85" y="43.18" smashed="yes" rot="R90"/>
-<element name="U$3" library="MRSDTeamB" package="TO220V" value="MIC29150/29300/29500VERTICAL" x="85.09" y="43.18" smashed="yes" rot="R90"/>
+<element name="U1" library="MRSDTeamB" package="TO220V" value="" x="54.61" y="43.18" rot="R90"/>
+<element name="U2" library="MRSDTeamB" package="TO220V" value="" x="69.85" y="43.18" rot="R90"/>
+<element name="U3" library="MRSDTeamB" package="TO220V" value="" x="85.09" y="43.18" rot="R90"/>
 <element name="BATT2" library="MRSDTeamB" package="CON_XT60_PCB_MOUNT" value="" x="41.91" y="11.43" rot="R90"/>
 <element name="BATT1" library="MRSDTeamB" package="CON_XT60_PCB_MOUNT" value="" x="31.75" y="11.43" rot="R90"/>
@@
 <contactref element="R4" pad="2"/>
 <contactref element="ACC1" pad="1"/>
-<contactref element="U$1" pad="3"/>
+<contactref element="U1" pad="3"/>
 <wire x1="60.96" y1="45.95" x2="60.96" y2="45.72" width="0.6096" layer="1"/>
 <wire x1="60.96" y1="45.72" x2="57.15" y2="45.72" width="0.6096" layer="1"/>
@@
 <contactref element="ACC2" pad="1"/>
 <contactref element="R5" pad="2"/>
-<contactref element="U$2" pad="3"/>
+<contactref element="U2" pad="3"/>
 <wire x1="76.2" y1="45.95" x2="72.62" y2="45.95" width="0.6096" layer="1"/>
 <wire x1="72.62" y1="45.95" x2="72.39" y2="45.72" width="0.6096" layer="1"/>
@@
 <contactref element="BATT2_W" pad="V-"/>
 <contactref element="BATT1_W" pad="V-"/>
-<contactref element="U$1" pad="2"/>
-<contactref element="U$2" pad="2"/>
-<contactref element="U$3" pad="2"/>
+<contactref element="U1" pad="2"/>
+<contactref element="U2" pad="2"/>
+<contactref element="U3" pad="2"/>
 <polygon width="0.8128" layer="16" isolate="0.8128">
 <vertex x="0.635" y="75.565"/>
@@
 <contactref element="ACC3" pad="1"/>
 <contactref element="R6" pad="2"/>
-<contactref element="U$3" pad="3"/>
+<contactref element="U3" pad="3"/>
 <wire x1="91.44" y1="45.95" x2="87.86" y2="45.95" width="0.6096" layer="1"/>
 <wire x1="87.86" y1="45.95" x2="87.63" y2="45.72" width="0.6096" layer="1"/>
@@
 <contactref element="F_BATT" pad="B3"/>
 <contactref element="F_BATT" pad="B4"/>
-<contactref element="U$1" pad="1"/>
-<contactref element="U$2" pad="1"/>
-<contactref element="U$3" pad="1"/>
+<contactref element="U1" pad="1"/>
+<contactref element="U2" pad="1"/>
+<contactref element="U3" pad="1"/>
 <contactref element="F_SERVO1" pad="A4"/>
 <contactref element="F_SERVO1" pad="A1"/>
