File: Eagle/PDM_simplified/PDM.brd (EAGLE design)
At the start: 50.5 x 63.5 mm, 24 parts

Commit message: Finalized PCB for fab
Parts:
- moved R7 1.91 mm to (33.7, 22.2)
- moved BATT 1.90 mm to (30.5, 10.2)
- moved C3 1.90 mm to (37.5, 10.8)
- moved R8 1.90 mm to (37.5, 15.9)
- moved D2 1.27 mm to (37.5, 5.71)
- moved R3 0.64 mm to (25.4, 45.7)
Routing:
- net GND: track 41.9 -> 46.8 mm
- net N$18: track 25.1 -> 21.0 mm
- net N$11: track 12.3 -> 13.0 mm
Changed lines of the file:
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@@
 <attribute name="NAME" x="15.875" y="47.625" size="1.27" layer="25" rot="R180"/>
 </element>
-<element name="R3" library="rcl" package="R1206" value="1K" x="26.035" y="45.72" smashed="yes" rot="R180">
-<attribute name="NAME" x="26.035" y="44.45" size="1.27" layer="25" rot="R180"/>
+<element name="R3" library="rcl" package="R1206" value="1K" x="25.4" y="45.72" smashed="yes" rot="R180">
+<attribute name="NAME" x="25.4" y="44.45" size="1.27" layer="25" rot="R180"/>
 </element>
 <element name="R4" library="rcl" package="R1206" value="1K" x="35.56" y="43.18" smashed="yes" rot="R180">
 <attribute name="NAME" x="35.56" y="41.91" size="1.27" layer="25" rot="R180"/>
 </element>
-<element name="R7" library="rcl" package="R1206" value="1.5K" x="31.75" y="22.225" rot="R90"/>
-<element name="R8" library="rcl" package="R1206" value="1K" x="37.465" y="13.97"/>
+<element name="R7" library="rcl" package="R1206" value="1.5K" x="33.655" y="22.225" rot="R90"/>
+<element name="R8" library="rcl" package="R1206" value="1K" x="37.465" y="15.875"/>
 <element name="C5" library="rcl" package="C1206K" value="10uF" x="29.21" y="34.29" smashed="yes" rot="R90">
 <attribute name="NAME" x="28.11" y="33.325" size="1.016" layer="25" rot="R90"/>
@@
 <attribute name="VALUE" x="15.24" y="1.905" size="1.27" layer="27"/>
 </element>
-<element name="D2" library="diode" package="SOD80C" value="3.3V" x="37.465" y="4.445" rot="R180"/>
+<element name="D2" library="diode" package="SOD80C" value="3.3V" x="37.465" y="5.715" rot="R180"/>
 <element name="DUE" library="con-molex" package="5566-2" value="" x="22.225" y="52.07">
 <attribute name="OC_NEWARK" value="unknown" x="106.045" y="-39.37" size="1.778" layer="27" display="off"/>
@@
 <element name="DUE_FUSE" library="MRSDTeamB" package="MINI_ATO" value="2A" x="22.225" y="27.94" rot="R180"/>
 <element name="SERVO_FUSE" library="MRSDTeamB" package="MINI_ATO" value="7.5A" x="10.795" y="27.94" rot="R180"/>
-<element name="C3" library="rcl" package="C1206K" value="10uF" x="37.465" y="8.89" rot="R180"/>
-<element name="BATT" library="MRSDTeamB" package="CON_XT60_PCB_MALE" value="" x="30.48" y="8.255" rot="R90"/>
+<element name="C3" library="rcl" package="C1206K" value="10uF" x="37.465" y="10.795" rot="R180"/>
+<element name="BATT" library="MRSDTeamB" package="CON_XT60_PCB_MALE" value="" x="30.48" y="10.16" rot="R90"/>
 </elements>
 <signals>
@@
 <contactref element="C1" pad="1"/>
 <polygon width="0.8128" layer="1" isolate="0.6096" thermals="no">
-<vertex x="19.685" y="30.48"/>
-<vertex x="19.685" y="48.895"/>
+<vertex x="20.32" y="30.48"/>
+<vertex x="20.32" y="49.53"/>
 <vertex x="20.955" y="50.165"/>
 <vertex x="23.495" y="50.165"/>
-<vertex x="24.765" y="48.895"/>
-<vertex x="24.765" y="31.115"/>
+<vertex x="24.13" y="49.53"/>
+<vertex x="24.13" y="30.48"/>
 </polygon>
 <contactref element="DUE_FUSE" pad="P$3"/>
@@
 </polygon>
 <polygon width="0.4064" layer="1" isolate="1.27" thermals="no">
-<vertex x="15.875" y="7.62"/>
-<vertex x="32.385" y="7.62"/>
-<vertex x="32.385" y="3.175"/>
-<vertex x="15.875" y="3.175"/>
+<vertex x="16.51" y="6.985"/>
+<vertex x="30.48" y="6.985"/>
+<vertex x="30.48" y="3.81"/>
+<vertex x="16.51" y="3.81"/>
 </polygon>
 <wire x1="33.655" y1="35.56" x2="37.465" y2="35.56" width="0.6096" layer="1"/>
@@
 <wire x1="43.025" y1="43.18" x2="43.025" y2="40.89" width="0.6096" layer="1"/>
 <wire x1="43.025" y1="40.89" x2="37.465" y2="35.33" width="0.6096" layer="1"/>
-<wire x1="36.043" y1="13.97" x2="36.043" y2="8.968" width="0.6096" layer="1"/>
-<wire x1="36.043" y1="8.968" x2="35.965" y2="8.89" width="0.6096" layer="1"/>
-<wire x1="35.965" y1="8.89" x2="35.965" y2="4.645" width="0.6096" layer="1"/>
-<wire x1="35.965" y1="4.645" x2="35.765" y2="4.445" width="0.6096" layer="1"/>
-<wire x1="35.765" y1="4.445" x2="30.69" y2="4.445" width="0.6096" layer="1"/>
-<wire x1="30.69" y1="4.445" x2="30.48" y2="4.655" width="0.6096" layer="1"/>
+<wire x1="36.043" y1="15.875" x2="36.043" y2="8.968" width="0.6096" layer="1"/>
+<wire x1="36.043" y1="8.968" x2="35.965" y2="10.795" width="0.6096" layer="1"/>
+<wire x1="35.965" y1="10.795" x2="35.965" y2="5.915" width="0.6096" layer="1"/>
+<wire x1="35.965" y1="5.915" x2="35.765" y2="5.715" width="0.6096" layer="1"/>
+<wire x1="35.765" y1="5.715" x2="30.69" y2="5.715" width="0.6096" layer="1"/>
+<wire x1="30.69" y1="5.715" x2="30.48" y2="6.56" width="0.6096" layer="1"/>
 </signal>
 <signal name="N$15">
@@
 <contactref element="C2" pad="+"/>
 <polygon width="0.6096" layer="1" isolate="0.8128" thermals="no">
-<vertex x="15.24" y="31.115"/>
-<vertex x="6.35" y="31.115"/>
-<vertex x="6.35" y="52.07"/>
+<vertex x="14.605" y="30.48"/>
+<vertex x="6.985" y="30.48"/>
+<vertex x="6.985" y="52.705"/>
 <vertex x="8.89" y="54.61"/>
 <vertex x="12.7" y="54.61"/>
-<vertex x="15.24" y="52.07"/>
+<vertex x="14.605" y="52.705"/>
 </polygon>
 <contactref element="SERVO_FUSE" pad="P$3"/>
@@
 <contactref element="R8" pad="2"/>
 <contactref element="D2" pad="C"/>
-<wire x1="38.735" y1="20.955" x2="31.75" y2="20.803" width="0.6096" layer="1"/>
+<wire x1="38.735" y1="20.955" x2="33.655" y2="20.803" width="0.6096" layer="1"/>
 <contactref element="C3" pad="1"/>
-<wire x1="38.735" y1="20.955" x2="38.735" y2="14.122" width="0.6096" layer="1"/>
-<wire x1="38.735" y1="14.122" x2="38.887" y2="13.97" width="0.6096" layer="1"/>
-<wire x1="38.887" y1="13.97" x2="38.887" y2="8.407" width="0.6096" layer="1"/>
-<wire x1="38.887" y1="8.407" x2="38.735" y2="8.255" width="0.6096" layer="1"/>
-<wire x1="38.735" y1="8.255" x2="38.735" y2="8.66" width="0.6096" layer="1"/>
-<wire x1="38.735" y1="8.66" x2="38.965" y2="8.89" width="0.6096" layer="1"/>
-<wire x1="38.965" y1="8.89" x2="38.965" y2="4.645" width="0.6096" layer="1"/>
-<wire x1="38.965" y1="4.645" x2="39.165" y2="4.445" width="0.6096" layer="1"/>
+<wire x1="38.735" y1="20.955" x2="38.735" y2="16.027" width="0.6096" layer="1"/>
+<wire x1="38.735" y1="16.027" x2="38.887" y2="15.875" width="0.6096" layer="1"/>
+<wire x1="38.887" y1="15.875" x2="38.887" y2="14.122" width="0.6096" layer="1"/>
+<wire x1="38.887" y1="14.122" x2="38.735" y2="11.43" width="0.6096" layer="1"/>
+<wire x1="38.735" y1="11.43" x2="38.735" y2="10.565" width="0.6096" layer="1"/>
+<wire x1="38.735" y1="10.565" x2="38.965" y2="10.795" width="0.6096" layer="1"/>
+<wire x1="38.965" y1="10.795" x2="38.965" y2="5.915" width="0.6096" layer="1"/>
+<wire x1="38.965" y1="5.915" x2="39.165" y2="5.715" width="0.6096" layer="1"/>
 </signal>
 <signal name="N$5">
@@
 <contactref element="LED3" pad="A"/>
 <contactref element="R3" pad="1"/>
-<wire x1="27.457" y1="45.72" x2="29.845" y2="45.72" width="0.6096" layer="1"/>
+<wire x1="26.822" y1="45.72" x2="29.845" y2="45.72" width="0.6096" layer="1"/>
 <via x="29.845" y="45.72" extent="1-16" drill="0.6" shape="square"/>
 <wire x1="29.845" y1="45.72" x2="30.48" y2="46.355" width="0.6096" layer="16"/>
@@
 <polygon width="0.8128" layer="1" isolate="0.6096" thermals="no">
 <vertex x="13.335" y="17.78"/>
-<vertex x="13.335" y="3.81"/>
-<vertex x="10.795" y="3.81"/>
-<vertex x="6.985" y="6.985"/>
-<vertex x="6.985" y="24.765"/>
+<vertex x="13.335" y="4.445"/>
+<vertex x="10.795" y="4.445"/>
+<vertex x="7.62" y="6.985"/>
+<vertex x="7.62" y="24.765"/>
 <vertex x="25.4" y="24.765"/>
-<vertex x="25.4" y="19.05"/>
-<vertex x="14.605" y="19.05"/>
+<vertex x="20.955" y="19.685"/>
+<vertex x="15.24" y="19.685"/>
 </polygon>
 <contactref element="BATT_FUSE" pad="P$3"/>
@@
 <wire x1="33.655" y1="33.02" x2="30.075" y2="33.02" width="0.6096" layer="1"/>
 <wire x1="30.075" y1="33.02" x2="29.21" y2="32.79" width="0.6096" layer="1"/>
-<wire x1="33.655" y1="24.13" x2="31.75" y2="23.647" width="0" layer="19" extent="1-1"/>
+<wire x1="33.655" y1="24.13" x2="33.655" y2="23.647" width="0" layer="19" extent="1-1"/>
 </signal>
 <signal name="N$2">
 <polygon width="0.8128" layer="1" isolate="0.6096" thermals="no">
-<vertex x="19.05" y="10.16"/>
-<vertex x="19.05" y="15.24"/>
-<vertex x="32.385" y="15.24"/>
-<vertex x="32.385" y="10.16"/>
+<vertex x="19.05" y="11.43"/>
+<vertex x="19.05" y="16.51"/>
+<vertex x="31.75" y="16.51"/>
+<vertex x="31.75" y="11.43"/>
 </polygon>
 <contactref element="BATT_FUSE" pad="P$2"/>
