Commit message: added joint state publisher to launch file and renamed foot locs to match planner defs

File: ROS/src/spacejockey/resources/spacejockey.urdf (robot description, URDF)
Before this commit: robot spacejockey, 8 links, 7 joints
Links:
- removed link base_link
- removed link front_seg
- removed link rear_seg
- added link center_foot; visual cylinder length=0.05 radius=0.2
- added link front_foot; visual cylinder length=0.04 radius=0.15
- added link rear_foot; visual cylinder length=0.04 radius=0.15
Joints:
- joint center_swivel: parent base_link -> center_foot
- joint fore_base_pitch: parent base_link -> center_foot
- joint front_pitch: child front_seg -> front_foot
- joint rear_pitch: child rear_seg -> rear_foot

Commit message: added camera transform to URDF

File: ROS/src/spacejockey/resources/spacejockey.urdf (robot description, URDF)
Before this commit: robot spacejockey, 8 links, 7 joints
Links:
- added link camera
Joints:
- added joint camera_fixed: type fixed, parent front_foot, child camera, origin xyz=.2 .05 .1 rpy=0 .3 0

Commit message: merged brian's URDF changes

File: ROS/src/spacejockey/resources/spacejockey.urdf (robot description, URDF)
Before this commit: robot spacejockey, 9 links, 8 joints
Links:
- removed link rear_foot
- added link back_foot; visual cylinder length=0.04 radius=0.15
- link aft_base_pole: geometry visual box size=.100 .032 .162
- link center_aft: geometry visual box size=.075 .095 .032
- link center_foot: geometry visual box size=.075 .095 .053
- link fore_base_pole: geometry visual box size=.100 .032 .162
Joints:
- joint aft_base_pitch: origin xyz=0 -.4 0 rpy=0 0 0 -> xyz=0 -.095 0 rpy=0 0 0
- joint center_swivel: origin xyz=0 -0.2 0 rpy=0 0 0 -> xyz=0 -0.0475 0 rpy=0 0 0
- joint fore_base_pitch: origin xyz=0 .2 0 rpy=0 0 0 -> xyz=0 .0475 0 rpy=0 0 0
- joint rear_pitch: child rear_foot -> back_foot

Commit message: added detach joint stubs to URDF file

File: ROS/src/spacejockey/resources/spacejockey.urdf (robot description, URDF)
Before this commit: robot flexible, 9 links, 8 joints
Links:
- removed link back_foot
- added link center_detach
- added link front_detach
- added link rear_detach
- added link rear_foot; visual cylinder length=0.04 radius=0.15
Joints:
- added joint center_attach: type prismatic, parent center_foot, child center_detach, origin xyz=0 0.0 0 rpy=0 0 0, limit lower=0 upper=0.006 effort=1000.0 velocity=0.5
- added joint front_attach: type prismatic, parent front_foot, child front_detach, origin xyz=0 0.0 0 rpy=0 0 0, limit lower=0 upper=0.006 effort=1000.0 velocity=0.5
- added joint rear_attach: type prismatic, parent rear_foot, child rear_detach, origin xyz=0 0.0 0 rpy=0 0 0, limit lower=0 upper=0.006 effort=1000.0 velocity=0.5
- joint rear_pitch: child back_foot -> rear_foot

Commit message: fixed joint order and urdf dimensions

File: ROS/src/spacejockey/resources/spacejockey.urdf (robot description, URDF)
Before this commit: robot flexible, 12 links, 11 joints
Links:
- removed link center_detach
- removed link front_detach
- removed link rear_detach
- added link center_seg; visual box size=.075 .095 .053
- added link front_seg; visual box size=.060 .095 .060
- added link rear_seg; visual box size=.060 .095 .060
- link aft_base_prism: geometry visual cylinder length=0.15 radius=.010
- link center_foot: geometry 
- link fore_base_prism: geometry visual cylinder length=0.15 radius=.010
- link front_foot: geometry 
- link rear_foot: geometry 
Joints:
- joint aft_base_pitch: origin xyz=0 -.095 0 rpy=0 0 0 -> xyz=0 -0.06985 0
- joint aft_extend: limit lower=0 upper=0.15 effort=1000.0 velocity=0.5 -> lower=0.19726 upper=0.27315 effort=1000.0 velocity=0.5
- joint camera_fixed: origin xyz=.2 .05 .1 rpy=0 .3 0 -> xyz=.06 .025 -.03 rpy=0 .3 0; parent front_foot -> front_seg
- joint center_attach: axis (none) -> 0 0 1; child center_detach -> center_seg; origin xyz=0 0.0 0 rpy=0 0 0 -> xyz=0 0 .050
- joint center_swivel: axis 0 0 -1 -> 0 0 1; origin xyz=0 -0.0475 0 rpy=0 0 0 -> (none); parent center_foot -> center_seg
- joint fore_base_pitch: origin xyz=0 .0475 0 rpy=0 0 0 -> xyz=0 0.06985 0; parent center_foot -> center_seg
- joint fore_extend: limit lower=0 upper=0.15 effort=1000.0 velocity=0.5 -> lower=0.19726 upper=0.27315 effort=1000.0 velocity=0.5
- joint front_attach: axis (none) -> 0 0 -1; child front_detach -> front_foot; origin xyz=0 0.0 0 rpy=0 0 0 -> xyz=0.00069 0 -0.04763; parent front_foot -> front_seg
- joint front_pitch: child front_foot -> front_seg; origin xyz=0.15 0 0 rpy=0 0 0 -> (none)
- joint rear_attach: axis (none) -> 0 0 -1; child rear_detach -> rear_foot; origin xyz=0 0.0 0 rpy=0 0 0 -> xyz=0.00069 0 -0.04763; parent rear_foot -> rear_seg
- joint rear_pitch: child rear_foot -> rear_seg; origin xyz=0.15 0 0 rpy=0 0 0 -> (none)

Commit message: fixed control_bridge joint ordering

File: ROS/src/spacejockey/resources/spacejockey.urdf (robot description, URDF)
Before this commit: robot Space Jockey, 12 links, 11 joints
Joints:
- joint center_attach: origin xyz=0 0 .050 -> xyz=0 0 .067

Commit message: reorganized urdf to match planner

File: ROS/src/spacejockey/resources/spacejockey.urdf (robot description, URDF)
Before this commit: robot Space Jockey, 12 links, 11 joints
Joints:
- joint center_attach: child center_seg -> center_aft
- joint center_swivel: child center_aft -> center_seg; parent center_seg -> center_aft

Commit message: Rewrote ROS side and control bridge

File: ROS/src/spacejockey/resources/spacejockey.urdf (robot description, URDF)
Before this commit: robot Space Jockey, 12 links, 11 joints
Joints:
- joint front_pitch: limit lower=-1.2 upper=1.2 effort=1000.0 velocity=0.5 -> lower=-.6 upper=.6 effort=1000.0 velocity=0.5
- joint rear_pitch: limit lower=-1.2 upper=1.2 effort=1000.0 velocity=0.5 -> lower=-.6 upper=.6 effort=1000.0 velocity=0.5

Commit message: fixed unused attach joints

File: ROS/src/spacejockey/resources/spacejockey.urdf (robot description, URDF)
Before this commit: robot Space Jockey, 12 links, 11 joints
Joints:
- joint front_attach: axis 0 0 -1 -> (none); limit lower=0 upper=0.006 effort=1000.0 velocity=0.5 -> (none); type prismatic -> fixed
- joint rear_attach: axis 0 0 -1 -> (none); limit lower=0 upper=0.006 effort=1000.0 velocity=0.5 -> (none); type prismatic -> fixed

Commit message: messin with frames

File: ROS/src/spacejockey/resources/spacejockey.urdf (robot description, URDF)
Before this commit: robot Space Jockey, 12 links, 11 joints
Links:
- added link robot
Joints:
- added joint base_fixed: type fixed, parent robot, child center_aft, origin xyz=0 0 .067
- joint center_attach: axis 0 0 1 -> 0 0 -1; child center_aft -> center_foot; origin xyz=0 0 .067 -> (none); parent center_foot -> robot

Commit message: updated URDF to be compliant with axis conventions see part 3 here: http://wiki.ros.org/Industrial/Tutorials/Create%20a%20URDF%20for%20an%20Industrial%20Robot

File: ROS/src/spacejockey/resources/spacejockey.urdf (robot description, URDF)
Before this commit: robot Space Jockey, 13 links, 12 joints
Links:
- link aft_base_pole: geometry visual box size=.162 .100 .032
- link center_aft: geometry visual box size=.095 .075 .032
- link center_seg: geometry visual box size=.095 .075 .053
- link fore_base_pole: geometry visual box size=.162 .100 .032
Joints:
- joint aft_base_pitch: axis -1 0 0 -> 0 1 0; origin xyz=0 -0.06985 0 -> xyz=-0.06985 0 0
- joint aft_extend: axis (none) -> -1 0 0; origin xyz=0 0.0 0 rpy=0 0 -1.57075 -> (none)
- joint fore_base_pitch: axis 1 0 0 -> 0 1 0; origin xyz=0 0.06985 0 -> xyz=0.06985 0 0
- joint fore_extend: origin xyz=0 0.0 0 rpy=0 0 1.57075 -> (none)
- joint front_pitch: axis 0 -1 0 -> 0 1 0
- joint rear_pitch: axis 0 -1 0 -> 0 1 0

Commit message: rolled planner stuff into main launch file

File: ROS/src/spacejockey/resources/spacejockey.urdf (robot description, URDF)
Before this commit: robot Space Jockey, 13 links, 12 joints
Links:
- link center_aft: geometry visual box size=.095 .075 .05
- link center_seg: geometry visual box size=.095 .075 .032

Commit message: joint vels

File: ROS/src/spacejockey/resources/spacejockey.urdf (robot description, URDF)
Before this commit: robot Space Jockey, 13 links, 12 joints
Joints:
- joint aft_base_pitch: limit lower=-.6 upper=.6 effort=1000.0 velocity=0.5 -> lower=-.6 upper=.6 effort=1000.0 velocity= 2.094
- joint aft_extend: limit lower=0.19726 upper=0.27315 effort=1000.0 velocity=0.5 -> lower=0.19726 upper=0.048 effort=1000.0 velocity=0.5
- joint center_attach: limit lower=0 upper=0.006 effort=1000.0 velocity=0.5 -> lower=0 upper=0.006 effort=1000.0 velocity=0. 2.094
- joint center_swivel: limit lower=-.8 upper=.8 effort=1000.0 velocity=0.5 -> lower=-.8 upper=.8 effort=1000.0 velocity= 2.094
- joint fore_base_pitch: limit lower=-.6 upper=.6 effort=1000.0 velocity=0.5 -> lower=-.6 upper=.6 effort=1000.0 velocity= 2.094
- joint fore_extend: limit lower=0.19726 upper=0.27315 effort=1000.0 velocity=0.5 -> lower=0.19726 upper=0.048 effort=1000.0 velocity=0.5
- joint front_pitch: limit lower=-.6 upper=.6 effort=1000.0 velocity=0.5 -> lower=-.6 upper=.6 effort=1000.0 velocity= 2.094
- joint rear_pitch: limit lower=-.6 upper=.6 effort=1000.0 velocity=0.5 -> lower=-.6 upper=.6 effort=1000.0 velocity= 2.094

Commit message: fixed syntax errors

File: ROS/src/spacejockey/resources/spacejockey.urdf (robot description, URDF)
Before this commit: robot Space Jockey, 13 links, 12 joints
Joints:
- joint aft_base_pitch: limit lower=-.6 upper=.6 effort=1000.0 velocity= 2.094 -> lower=-.6 upper=.6 effort=1000.0 velocity=2.094
- joint center_attach: limit lower=0 upper=0.006 effort=1000.0 velocity=0. 2.094 -> lower=0 upper=0.006 effort=1000.0 velocity=1.0
- joint center_swivel: limit lower=-.8 upper=.8 effort=1000.0 velocity= 2.094 -> lower=-.8 upper=.8 effort=1000.0 velocity=2.094
- joint fore_base_pitch: limit lower=-.6 upper=.6 effort=1000.0 velocity= 2.094 -> lower=-.6 upper=.6 effort=1000.0 velocity=2.094
- joint front_pitch: limit lower=-.6 upper=.6 effort=1000.0 velocity= 2.094 -> lower=-.6 upper=.6 effort=1000.0 velocity=2.094
- joint rear_pitch: limit lower=-.6 upper=.6 effort=1000.0 velocity= 2.094 -> lower=-.6 upper=.6 effort=1000.0 velocity=2.094
- joint robot_rot: limit lower=-3.15 upper=3.15 effort=1000.0 velocity=0.5 -> lower=-3.15 upper=3.15 effort=1000.0 velocity=2.094

Commit message: demo code

File: ROS/src/spacejockey/resources/spacejockey.urdf (robot description, URDF)
Before this commit: robot Space Jockey, 13 links, 12 joints
Joints:
- joint aft_extend: limit lower=0.19726 upper=0.048 effort=1000.0 velocity=0.5 -> lower=0.1902 upper=0.2781 effort=1000.0 velocity=0.048
- joint camera_fixed: origin xyz=.06 .025 -.03 rpy=0 .3 0 -> xyz=.06 -.025 -.03 rpy=0 2.3562 0
- joint fore_extend: limit lower=0.19726 upper=0.048 effort=1000.0 velocity=0.5 -> lower=0.1902 upper=0.2781 effort=1000.0 velocity=0.048

Commit message: Camera URDF
Corrected camera in urdf

File: ROS/src/spacejockey/resources/spacejockey.urdf (robot description, URDF)
Before this commit: robot Space Jockey, 13 links, 12 joints
Joints:
- joint camera_fixed: origin xyz=.06 -.025 -.03 rpy=0 2.3562 0 -> xyz=.082 .019 -.009 rpy=0 2.3562 0

Commit message: Recalibrated feet, swivel joint (was way off)
Fixes #20

File: ROS/src/spacejockey/resources/spacejockey.urdf (robot description, URDF)
Before this commit: robot Space Jockey, 13 links, 12 joints
Joints:
- joint center_swivel: limit lower=-.8 upper=.8 effort=1000.0 velocity=2.094 -> lower=-.35 upper=.35 effort=1000.0 velocity=2.094
- joint front_pitch: limit lower=-.6 upper=.6 effort=1000.0 velocity=2.094 -> lower=-.52 upper=.78 effort=1000.0 velocity=2.094

Commit message: Updated calibration

File: ROS/src/spacejockey/resources/spacejockey.urdf (robot description, URDF)
Before this commit: robot Space Jockey, 13 links, 12 joints
Joints:
- joint front_pitch: limit lower=-.52 upper=.78 effort=1000.0 velocity=2.094 -> lower=-.70 upper=.873 effort=1000.0 velocity=2.094

Commit message: Calibration Update

File: ROS/src/spacejockey/resources/spacejockey.urdf (robot description, URDF)
Before this commit: robot Space Jockey, 13 links, 12 joints
Joints:
- joint aft_base_pitch: limit lower=-.6 upper=.6 effort=1000.0 velocity=2.094 -> lower=-.524 upper=.524 effort=1000.0 velocity=2.094
- joint center_swivel: limit lower=-.35 upper=.35 effort=1000.0 velocity=2.094 -> lower=-.436 upper=.436 effort=1000.0 velocity=2.094
- joint fore_base_pitch: limit lower=-.6 upper=.6 effort=1000.0 velocity=2.094 -> lower=-.524 upper=.524 effort=1000.0 velocity=2.094
- joint front_pitch: limit lower=-.70 upper=.873 effort=1000.0 velocity=2.094 -> lower=-.785 upper=.785 effort=1000.0 velocity=2.094
- joint rear_pitch: limit lower=-.6 upper=.6 effort=1000.0 velocity=2.094 -> lower=-.785 upper=.785 effort=1000.0 velocity=2.094
